Commit message: Fixed frames for the whole system, organized structure a bit

File: AkulaPackageROS2/model/akula_general.xacro (robot description, xacro)
@@ -116,16 +116,15 @@
   </xacro:macro>
   <!-- - - - - - - - - - - - Basler camera - - - - - - - - - - - -->
-<xacro:macro name="camera" params="parent camera_name *origin">
-  <joint name="${camera_name}_base_mount_joint" type="fixed">
-    <xacro:insert_block name="origin"/>
-    <parent link="${parent}_base"/>
-    <child link="${camera_name}"/>
-  </joint>
-  <link name="${camera_name}">
+<xacro:macro name="basler" params="parent *origin">
+  <joint name="basler_base_mount_joint" type="fixed">
+      <xacro:insert_block name="origin"/>
+      <parent link="${parent}_base"/>
+      <child link="basler"/>
+    </joint>
+  <link name="basler">
     <visual>
-      <!-- z is zero for now -->
-      <origin rpy="0 1.57 0" xyz="0 0 0"/>
+      <origin rpy="1.57 0 1.57" xyz="-0.05 0 0"/>
       <geometry>
-        <cylinder radius="0.01" length="0.1" />
+        <box size="0.03 0.03 0.1"/>
       </geometry>
       <material name="AKULA/LightGrey" />
